File: lunchbeat-PCB-hardware/lunchbeat-PCB-kicadproject/lunchbeat-PCB.kicad_pcb (KiCad board)
At the start: 2 copper layers, 140 x 65 mm, 70 parts, among them J1 AUDIO OUT, J2 SYNC IN, SW1 SW-PW, U1 LM358N, U2 ATMEGA328P, U3 74595, U4 7805

Commit message: kit1
Parts:
- added Ref**: bla, buran-lunch-17x32-med, F.Cu at (98.2, 78.3)
- added Ref**: Val**, lunchdeska1-l20, F.Cu at (155.0, 94.5)
Connections:
- net N-000008 renamed /batvcc
Routing:
- net /LATCH: track 77.0 -> 79.6 mm
- net /DATA: track 124.6 -> 122.5 mm
- net /CLOCK: track 79.8 -> 78.9 mm
Other:
- outline, holes or cut-outs redrawn
- net class Default: via_dia 1.5 -> 1.8; via_drill 0.6 -> 0.7
- net class batt: via_dia 1.5 -> 1.8; via_drill 0.6 -> 0.7
- net class gnd: via_dia 1.5 -> 1.8; via_drill 0.6 -> 0.7
- net class vcc: via_dia 1.5 -> 1.8; via_drill 0.6 -> 0.7
