File: lunchbeat-PCB-hardware/lunchbeat-PCB-kicadproject/lunchbeat-PCB.sch (KiCad schematic (older format))
At the start: 62 parts, among them J1 AUDIO OUT, J2 SYNC IN, SW1 SW-PW, U1 LM358N, U2 ATMEGA328P, U3 74595, U4 7805

Commit message: kit1
Connections:
- net labels added: batvcc
Changed lines of the file:
@@
 	10450 5950 10450 6350
 Connection ~ 10450 6350
+Text Label 7400 5450 3    39   ~ 0
+batvcc
 $EndSCHEMATC
